File: lets play together/board.brd (EAGLE design)
At the start: 20 x 98.5 mm, 23 parts, among them IC1 TL074P, SW1 SUB-MINI, SW2 SUB-MINI, SW3 JS202011CQN

Commit message: Let's play together rev0
Parts:
- removed SW2: SUB-MINI, switch:TL3XPO
- moved SW1 6.26 mm to (10.0, 61.5), turned to 270 degrees
- moved ANALOG 6.00 mm to (4.50, 7.00)
- moved D1 6.00 mm to (12.5, 74.0)
- moved D2 6.00 mm to (5.50, 74.0)
- moved JP2 6.00 mm to (3.00, 84.0)
- moved L1 6.00 mm to (9.00, 74.0)
- moved L2 6.00 mm to (2.00, 74.0)
- moved VR1 6.00 mm to (10.0, 89.5)
- moved LED1 5.39 mm to (4.50, 17.0), turned to 0 degrees
- moved JP1 5.00 mm to (16.5, 75.0)
Connections:
- removed net D12: JP3.10, SW1.2
- net D10: now also SW1.2; no longer SW2.2
- net GND: no longer SW2.1
Routing:
- net D12: track 22.0 -> 0.00 mm
- net +12V: track 58.3 -> 51.7 mm
- net A0: track 55.0 -> 49.0 mm
- net -12V: track 35.4 -> 29.4 mm
- net VCC: track 66.1 -> 60.1 mm
- net N$8: track 3.10 -> 9.07 mm
- net D3: track 26.2 -> 30.3 mm
- net D10: track 14.0 -> 11.8 mm
- net N$1: track 10.0 -> 11.0 mm
- net CLOCK: track 90.1 -> 89.5 mm
Other:
- board size 20 x 98.5 mm -> 20 x 92.5 mm
