File: lets play together/board.sch (EAGLE design)
At the start: 23 parts, among them IC1 TL074P, SW1 SUB-MINI, SW2 SUB-MINI, SW3 JS202011CQN

Commit message: Let's play together rev0
Parts:
- removed SW2: SUB-MINI, switch:TL36PO
Connections:
- removed net D12: JP3.D12, SW1.P
- net D10: now also SW1.P; no longer SW2.P
- net GND: no longer SW2.O
Other:
- moved on the sheet: SW1
Changed lines of the file:
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@@
 </part>
 <part name="GND3" library="supply1" library_urn="urn:adsk.eagle:library:371" deviceset="GND" device=""/>
-<part name="GND5" library="supply1" library_urn="urn:adsk.eagle:library:371" deviceset="GND" device=""/>
 <part name="GND2" library="supply1" library_urn="urn:adsk.eagle:library:371" deviceset="GND" device=""/>
 <part name="JP2" library="jumper" library_urn="urn:adsk.eagle:library:252" deviceset="JP1E" device="" package3d_urn="urn:adsk.eagle:package:15455/1">
@@
 <attribute name="OC_FARNELL" value="1248140"/>
 </part>
-<part name="SW1" library="switch" library_urn="urn:adsk.eagle:library:380" deviceset="TL36PO" device="" package3d_urn="urn:adsk.eagle:package:27745/1" value="SUB-MINI">
-<attribute name="MF" value=""/>
-<attribute name="MPN" value=""/>
-<attribute name="OC_FARNELL" value="unknown"/>
-</part>
 <part name="MIDI" library="MusicThingModular" deviceset="THONKI-STEREO" device="">
 <attribute name="MF" value=""/>
@@
 <part name="P+2" library="supply1" library_urn="urn:adsk.eagle:library:371" deviceset="+12V" device=""/>
 <part name="GND6" library="supply1" library_urn="urn:adsk.eagle:library:371" deviceset="GND" device=""/>
-<part name="SW2" library="switch" library_urn="urn:adsk.eagle:library:380" deviceset="TL36PO" device="" package3d_urn="urn:adsk.eagle:package:27745/1" value="SUB-MINI">
+<part name="SW1" library="switch" library_urn="urn:adsk.eagle:library:380" deviceset="TL36PO" device="" package3d_urn="urn:adsk.eagle:package:27745/1" value="SUB-MINI">
 <attribute name="MF" value=""/>
 <attribute name="MPN" value=""/>
@@
 <attribute name="VALUE" x="114.3" y="53.34" size="1.778" layer="96"/>
 </instance>
-<instance part="GND5" gate="1" x="33.02" y="76.2" smashed="yes">
-<attribute name="VALUE" x="30.48" y="73.66" size="1.778" layer="96"/>
-</instance>
 <instance part="IC1" gate="A" x="119.38" y="27.94" smashed="yes">
 <attribute name="NAME" x="121.92" y="31.115" size="1.778" layer="95"/>
@@
 <attribute name="MPN" x="160.02" y="93.98" size="1.778" layer="96" display="off"/>
 </instance>
-<instance part="SW1" gate="BEF1" x="40.64" y="83.82" smashed="yes" rot="R90">
-<attribute name="NAME" x="43.18" y="88.9" size="1.778" layer="95" rot="R180"/>
-<attribute name="OC_FARNELL" x="40.64" y="83.82" size="1.778" layer="96" display="off"/>
-<attribute name="MF" x="40.64" y="83.82" size="1.778" layer="96" display="off"/>
-<attribute name="MPN" x="40.64" y="83.82" size="1.778" layer="96" display="off"/>
-</instance>
 <instance part="MIDI" gate="G$1" x="175.26" y="33.02" smashed="yes" rot="R180">
 <attribute name="NAME" x="180.34" y="29.972" size="1.778" layer="95" rot="R180"/>
@@
 <attribute name="VALUE" x="30.48" y="58.42" size="1.778" layer="96"/>
 </instance>
-<instance part="SW2" gate="BEF1" x="40.64" y="68.58" smashed="yes" rot="R90">
-<attribute name="NAME" x="43.18" y="73.66" size="1.778" layer="95" rot="R180"/>
-<attribute name="OC_FARNELL" x="40.64" y="68.58" size="1.778" layer="96" display="off"/>
-<attribute name="MF" x="40.64" y="68.58" size="1.778" layer="96" display="off"/>
-<attribute name="MPN" x="40.64" y="68.58" size="1.778" layer="96" display="off"/>
+<instance part="SW1" gate="BEF1" x="40.64" y="73.66" smashed="yes" rot="R90">
+<attribute name="NAME" x="43.18" y="78.74" size="1.778" layer="95" rot="R180"/>
+<attribute name="OC_FARNELL" x="40.64" y="73.66" size="1.778" layer="96" display="off"/>
+<attribute name="MF" x="40.64" y="73.66" size="1.778" layer="96" display="off"/>
+<attribute name="MPN" x="40.64" y="73.66" size="1.778" layer="96" display="off"/>
 </instance>
 </instances>
@@
 </segment>
 <segment>
-<wire x1="35.56" y1="81.28" x2="33.02" y2="81.28" width="0.1524" layer="91"/>
-<wire x1="33.02" y1="81.28" x2="33.02" y2="78.74" width="0.1524" layer="91"/>
-<pinref part="GND5" gate="1" pin="GND"/>
-<pinref part="SW1" gate="BEF1" pin="O"/>
-</segment>
-<segment>
 <pinref part="IC1" gate="B" pin="+IN"/>
 <wire x1="111.76" y1="15.24" x2="104.14" y2="15.24" width="0.1524" layer="91"/>
@@
 </segment>
 <segment>
-<wire x1="35.56" y1="66.04" x2="33.02" y2="66.04" width="0.1524" layer="91"/>
-<wire x1="33.02" y1="66.04" x2="33.02" y2="63.5" width="0.1524" layer="91"/>
+<wire x1="35.56" y1="71.12" x2="33.02" y2="71.12" width="0.1524" layer="91"/>
+<wire x1="33.02" y1="71.12" x2="33.02" y2="63.5" width="0.1524" layer="91"/>
 <pinref part="GND6" gate="1" pin="GND"/>
-<pinref part="SW2" gate="BEF1" pin="O"/>
+<pinref part="SW1" gate="BEF1" pin="O"/>
 </segment>
 </net>
@@
 </segment>
 <segment>
-<wire x1="45.72" y1="68.58" x2="48.26" y2="68.58" width="0.1524" layer="91"/>
-<label x="48.26" y="68.58" size="1.778" layer="95" xref="yes"/>
-<pinref part="SW2" gate="BEF1" pin="P"/>
+<wire x1="45.72" y1="73.66" x2="48.26" y2="73.66" width="0.1524" layer="91"/>
+<label x="48.26" y="73.66" size="1.778" layer="95" xref="yes"/>
+<pinref part="SW1" gate="BEF1" pin="P"/>
 </segment>
 </net>
@@
 </segment>
 </net>
-<net name="D12" class="0">
-<segment>
-<pinref part="JP3" gate="G$1" pin="D12"/>
-<wire x1="93.98" y1="63.5" x2="96.52" y2="63.5" width="0.1524" layer="91"/>
-<label x="96.52" y="63.5" size="1.778" layer="95" xref="yes"/>
-</segment>
-<segment>
-<wire x1="45.72" y1="83.82" x2="48.26" y2="83.82" width="0.1524" layer="91"/>
-<label x="48.26" y="83.82" size="1.778" layer="95" xref="yes"/>
-<pinref part="SW1" gate="BEF1" pin="P"/>
-</segment>
-</net>
